File: stenomod-15L.kicad_pcb (KiCad board)
At the start: 2 copper layers, 124.5 x 80 mm, 37 parts

Commit message: more text on the board
Other:
- board text added: "Adafruit Metro Mini goes here"
- board text added: "Licensed under CERN OHL v.1.2"
Changed lines of the file:
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@@
     (area 76.149999 52.019999 200.710001 132.475)
     (thickness 1.6)
-    (drawings 17)
+    (drawings 19)
     (tracks 247)
     (zones 0)
@@
       (padsonsilk false)
       (subtractmaskfromsilk false)
-      (outputformat 1)
+      (outputformat 4)
       (mirror false)
-      (drillshape 1)
+      (drillshape 0)
       (scaleselection 1)
       (outputdirectory ""))
@@
     )
   )
+  (gr_text "Adafruit Metro Mini goes here" (at 87.63 74.295 90) (layer F.SilkS)
+    (effects (font (size 1.5 1.5) (thickness 0.3)))
+  )
+  (gr_text "Licensed under\nCERN OHL v.1.2" (at 88.265 107.315) (layer F.SilkS)
+    (effects (font (size 1.5 1.5) (thickness 0.3)))
+  )
   (gr_text 11 (at 99.06 62.23) (layer F.SilkS)
